Commit message: update link_chassis2

File: urdf/gazebo.xacro (robot description, xacro)
@@ -2,5 +2,5 @@
 <robot name="m2wr" xmlns:xacro="https://www.ros.org/wiki/xacro" >
   <!-- Define color for robot parts -->
-  <gazebo reference="link_chassis">
+  <gazebo reference="link_chassis_rb3">
     <material>Gazebo/Orange</material>
   </gazebo>
@@ -26,5 +26,5 @@
       <odometryTopic>robot3us/odom</odometryTopic>
       <odometryFrame>robor3us/odom</odometryFrame>
-      <robotBaseFrame>link_chassis</robotBaseFrame>
+      <robotBaseFrame>link_chassis_rb3</robotBaseFrame>
     </plugin>
   </gazebo>

File: urdf/m2wr.xacro (robot description, xacro)
@@ -12,5 +12,5 @@
   <xacro:include filename="$(find robot3us_sim)/urdf/macro.xacro" />
   <!-- Defining link chassis -->
-  <link name="link_chassis">
+  <link name="link_chassis_rb3">
     <!-- pose and inertial -->
     <pose>0 0 0.1 0 0 0</pose>
@@ -179,20 +179,20 @@
   <joint name="joint_sensor_laser" type="fixed">
     <origin xyz="0.15 0 0.05" rpy="0 0 0"/>
-    <parent link="link_chassis"/>
+    <parent link="link_chassis_rb3"/>
     <child link="sensor_laser"/>
   </joint>
    <joint name="joint_sensor_us_front" type="fixed">
     <origin xyz="0.25 0 0.02" rpy="0 0 0"/>
-    <parent link="link_chassis"/>
+    <parent link="link_chassis_rb3"/>
     <child link="sensor_us_link_front"/>
   </joint>
    <joint name="joint_sensor_us_right" type="fixed">
     <origin xyz="0.15 0.15 0" rpy="0 0 1.57"/>
-    <parent link="link_chassis"/>
+    <parent link="link_chassis_rb3"/>
     <child link="sensor_us_link_right"/>
   </joint>
    <joint name="joint_sensor_us_left" type="fixed">
     <origin xyz="0.15 -0.15 0" rpy="0 0 -1.57"/>
-    <parent link="link_chassis"/>
+    <parent link="link_chassis_rb3"/>
     <child link="sensor_us_link_left"/>
   </joint>

File: urdf/macro.xacro (robot description, xacro)
@@ -36,5 +36,5 @@
         <origin rpy="0 0 0" xyz="${origin_xyz}"/>
         <child link="${child}"/>
-        <parent link="link_chassis"/>
+        <parent link="link_chassis_rb3"/>
         <axis rpy="0 0 0" xyz="0 1 0"/>
         <limit effort="10000" velocity="1000"/>
