Commit message: update_us_urdf_el3007

File: urdf/m2wr.xacro (robot description, xacro)
@@ -127,30 +127,30 @@
     </collision>
 </link>
+<link name="sensor_us_link_right">
+    <collision>
+      <origin xyz="0 0 0" rpy="0 0 0"/>
+      <geometry>
+        <box size="0.01 0.01 0.01"/>
+      </geometry>
+    </collision>
+    <visual>
+      <origin xyz="0 0 0" rpy="0 0 0"/>
+      <geometry>
+        <box size="0.01 0.01 0.01"/>
+      </geometry>
+    </visual>
+    <inertial>
+      <mass value="1e-5" />
+      <origin xyz="0 0 0" rpy="0 0 0"/>
+      <inertia ixx="1e-6" ixy="0" ixz="0" iyy="1e-6" iyz="0" izz="1e-6" />
+    </inertial>
+    <collision>
+      <origin xyz="0 0 0" rpy="0 0 0"/>
+      <geometry>
+      <box size="0.01 0.01 0.01"/>
+      </geometry>
+    </collision>
+</link>
 <link name="sensor_us_link_left">
-    <collision>
-      <origin xyz="0 0 0" rpy="0 0 0"/>
-      <geometry>
-        <box size="0.01 0.01 0.01"/>
-      </geometry>
-    </collision>
-    <visual>
-      <origin xyz="0 0 0" rpy="0 0 0"/>
-      <geometry>
-        <box size="0.01 0.01 0.01"/>
-      </geometry>
-    </visual>
-    <inertial>
-      <mass value="1e-5" />
-      <origin xyz="0 0 0" rpy="0 0 0"/>
-      <inertia ixx="1e-6" ixy="0" ixz="0" iyy="1e-6" iyz="0" izz="1e-6" />
-    </inertial>
-    <collision>
-      <origin xyz="0 0 0" rpy="0 0 0"/>
-      <geometry>
-      <box size="0.01 0.01 0.01"/>
-      </geometry>
-    </collision>
-</link>
-<link name="sensor_us_link_right">
     <collision>
       <origin xyz="0 0 0" rpy="0 0 0"/>
@@ -187,13 +187,13 @@
     <child link="sensor_us_link_front"/>
   </joint>
-   <joint name="joint_sensor_us_right" type="fixed">
+   <joint name="joint_sensor_us_left" type="fixed">
     <origin xyz="0.15 0.15 0" rpy="0 0 1.57"/>
     <parent link="link_chassis_rb3"/>
-    <child link="sensor_us_link_right"/>
+    <child link="sensor_us_link_left"/>
   </joint>
-   <joint name="joint_sensor_us_left" type="fixed">
+   <joint name="joint_sensor_us_right" type="fixed">
     <origin xyz="0.15 -0.15 0" rpy="0 0 -1.57"/>
     <parent link="link_chassis_rb3"/>
-    <child link="sensor_us_link_left"/>
+    <child link="sensor_us_link_right"/>
   </joint>
   <gazebo reference="sensor_us_link_front">
@@ -234,5 +234,5 @@
    </sensor>
    </gazebo>
-   <gazebo reference="sensor_us_link_left">
+   <gazebo reference="sensor_us_link_right">
    <sensor type="ray" name="TeraRanger">
       <pose>0 0 0 0 0 0</pose>
@@ -265,5 +265,5 @@
          <updateRate>50</updateRate>
          <topicName>us_sensor_right</topicName>
-         <frameName>sensor_us_link_left</frameName>
+         <frameName>sensor_us_link_right</frameName>
          <radiation>SONAR</radiation>
          <fov>0.2967</fov>
@@ -271,5 +271,5 @@
    </sensor>
    </gazebo>
-   <gazebo reference="sensor_us_link_right">
+   <gazebo reference="sensor_us_link_left">
    <sensor type="ray" name="TeraRanger">
       <pose>0 0 0 0 0 0</pose>
@@ -302,5 +302,5 @@
          <updateRate>50</updateRate>
          <topicName>us_sensor_left</topicName>
-         <frameName>sensor_us_link_right</frameName>
+         <frameName>sensor_us_link_left</frameName>
          <radiation>SONAR</radiation>
          <fov>0.2967</fov>
